Commit message: add urdf folder based on https://github.com/elephantrobotics/mycobot_ros/pull/48

File: urdf/mycobot/mycobot.gazebo.xacro (robot description, xacro)
@@ -2,5 +2,5 @@
 <robot  xmlns:xacro="http://www.ros.org/wiki/xacro" name="mycobot" >
   <xacro:arg name="robot_namespace" default="" />
-  <xacro:include filename="$(find mycobot_description)/urdf/mycobot/mycobot.urdf.xacro" />
+  <xacro:include filename="$(find tork_moveit_tutorial)/urdf/mycobot/mycobot.urdf.xacro" />
   <gazebo>
     <plugin name="gazebo_ros_control" filename="libgazebo_ros_control.so">

File: urdf/mycobot/mycobot.urdf.xacro (robot description, xacro)
@@ -1,5 +1,5 @@
 <?xml version="1.0"?>
 <robot  xmlns:xacro="http://www.ros.org/wiki/xacro" name="mycobot" >
-  <xacro:include filename="$(find mycobot_description)/urdf/common.xacro" />
+  <xacro:include filename="$(find tork_moveit_tutorial)/urdf/common.xacro" />
   <link name="link1">
     <inertial>
@@ -10,5 +10,5 @@
     <visual>
       <geometry>
-       <mesh filename="package://mycobot_description/urdf/mycobot/mesh/link1.dae"/>
+       <mesh filename="package://tork_moveit_tutorial/urdf/mycobot/mesh/link1.dae"/>
       </geometry>
       <origin xyz = "0.0 0 0 " rpy = " 0 0 -${pi/2}"/>
@@ -16,5 +16,5 @@
     <collision>
       <geometry>
-       <mesh filename="package://mycobot_description/urdf/mycobot/mesh/link1.dae"/>
+       <mesh filename="package://tork_moveit_tutorial/urdf/mycobot/mesh/link1.dae"/>
         </geometry>
         <origin xyz = "0.0 0 0 " rpy = " 0 0 -${pi/2}"/>
@@ -29,5 +29,5 @@
     <visual>
       <geometry>
-       <mesh filename="package://mycobot_description/urdf/mycobot/mesh/link2.dae"/>
+       <mesh filename="package://tork_moveit_tutorial/urdf/mycobot/mesh/link2.dae"/>
       </geometry>
       <origin xyz = "0.0 0 -0.06096 " rpy = " 0 0 -${pi/2}"/>
@@ -35,5 +35,5 @@
     <collision>
      <geometry>
-       <mesh filename="package://mycobot_description/urdf/mycobot/mesh/link2.dae"/>
+       <mesh filename="package://tork_moveit_tutorial/urdf/mycobot/mesh/link2.dae"/>
       </geometry>
       <origin xyz = "0.0 0 -0.06096 " rpy = " 0 0 -${pi/2}"/>
@@ -48,5 +48,5 @@
     <visual>
       <geometry>
-       <mesh filename="package://mycobot_description/urdf/mycobot/mesh/link3.dae"/>
+       <mesh filename="package://tork_moveit_tutorial/urdf/mycobot/mesh/link3.dae"/>
       </geometry>
     <origin xyz = "0.0 0 0.03256 " rpy = " 0 -${pi/2} 0"/>
@@ -54,5 +54,5 @@
     <collision>
       <geometry>
-       <mesh filename="package://mycobot_description/urdf/mycobot/mesh/link3.dae"/>
+       <mesh filename="package://tork_moveit_tutorial/urdf/mycobot/mesh/link3.dae"/>
       </geometry>
       <origin xyz = "0.0 0 0.03256 " rpy = " 0 -${pi/2} 0"/>
@@ -68,5 +68,5 @@
       <geometry>
        <!--- 0.0 0 -0.04 -->
-       <mesh filename="package://mycobot_description/urdf/mycobot/mesh/link4.dae"/>
+       <mesh filename="package://tork_moveit_tutorial/urdf/mycobot/mesh/link4.dae"/>
       </geometry>
       <origin xyz = "0.0 0 0.03056 " rpy = " 0 -${pi/2} 0"/>
@@ -75,5 +75,5 @@
       <geometry>
        <!--- 0.0 0 -0.04 -->
-       <mesh filename="package://mycobot_description/urdf/mycobot/mesh/link4.dae"/>
+       <mesh filename="package://tork_moveit_tutorial/urdf/mycobot/mesh/link4.dae"/>
       </geometry>
       <origin xyz = "0.0 0 0.03056 " rpy = " 0 -${pi/2} 0"/>
@@ -89,5 +89,5 @@
       <geometry>
        <!--- 0.0 0 -0.04 -->
-       <mesh filename="package://mycobot_description/urdf/mycobot/mesh/link5.dae"/>
+       <mesh filename="package://tork_moveit_tutorial/urdf/mycobot/mesh/link5.dae"/>
       </geometry>
     <origin xyz = "0.0 0 -0.03356 " rpy = " -${pi/2} 0 0"/>
@@ -96,5 +96,5 @@
        <geometry>
        <!--- 0.0 0 -0.04 -->
-       <mesh filename="package://mycobot_description/urdf/mycobot/mesh/link5.dae"/>
+       <mesh filename="package://tork_moveit_tutorial/urdf/mycobot/mesh/link5.dae"/>
       </geometry>
       <origin xyz = "0.0 0 -0.03356 " rpy = " -${pi/2} 0 0"/>
@@ -110,5 +110,5 @@
       <geometry>
        <!--- 0.0 0 -0.04 -->
-       <mesh filename="package://mycobot_description/urdf/mycobot/mesh/link6.dae"/>
+       <mesh filename="package://tork_moveit_tutorial/urdf/mycobot/mesh/link6.dae"/>
       </geometry>
     <origin xyz = "0 0.00 -0.038 " rpy = " 0 0 0"/>
@@ -117,5 +117,5 @@
       <geometry>
        <!--- 0.0 0 -0.04 -->
-       <mesh filename="package://mycobot_description/urdf/mycobot/mesh/link6.dae"/>
+       <mesh filename="package://tork_moveit_tutorial/urdf/mycobot/mesh/link6.dae"/>
       </geometry>
     <origin xyz = "0 0.00 -0.038 " rpy = " 0 0 0"/>
@@ -131,5 +131,5 @@
       <geometry>
        <!--- 0.0 0 -0.04 -->
-       <mesh filename="package://mycobot_description/urdf/mycobot/mesh/link7.dae"/>
+       <mesh filename="package://tork_moveit_tutorial/urdf/mycobot/mesh/link7.dae"/>
       </geometry>
     <origin xyz = "0.0 0 -0.012 " rpy = " 0 0 0"/>
@@ -138,5 +138,5 @@
       <geometry>
        <!--- 0.0 0 -0.04 -->
-       <mesh filename="package://mycobot_description/urdf/mycobot/mesh/link7.dae"/>
+       <mesh filename="package://tork_moveit_tutorial/urdf/mycobot/mesh/link7.dae"/>
       </geometry>
     <origin xyz = "0.0 0 -0.012 " rpy = " 0 0 0"/>

File: urdf/mycobot/mycobot_with_vision.urdf (robot description, URDF)
Before this commit: robot mycobot_ai, 8 links, 7 joints
Links:
- link env: geometry visual mesh filename=package://tork_moveit_tutorial/urdf/mycobot/suit_env.dae
- link joint1: geometry collision mesh filename=package://tork_moveit_tutorial/urdf/mycobot/joint1.dae; visual mesh filename=package://tork_moveit_tutorial/urdf/mycobot/joint1.dae
- link joint2: geometry collision mesh filename=package://tork_moveit_tutorial/urdf/mycobot/joint2.dae; visual mesh filename=package://tork_moveit_tutorial/urdf/mycobot/joint2.dae
- link joint3: geometry collision mesh filename=package://tork_moveit_tutorial/urdf/mycobot/joint3.dae; visual mesh filename=package://tork_moveit_tutorial/urdf/mycobot/joint3.dae
- link joint4: geometry collision mesh filename=package://tork_moveit_tutorial/urdf/mycobot/joint4.dae; visual mesh filename=package://tork_moveit_tutorial/urdf/mycobot/joint4.dae
- link joint5: geometry collision mesh filename=package://tork_moveit_tutorial/urdf/mycobot/joint5.dae; visual mesh filename=package://tork_moveit_tutorial/urdf/mycobot/joint5.dae
- link joint6: geometry collision mesh filename=package://tork_moveit_tutorial/urdf/mycobot/joint6.dae; visual mesh filename=package://tork_moveit_tutorial/urdf/mycobot/joint6.dae
- link joint6_flange: geometry collision mesh filename=package://tork_moveit_tutorial/urdf/mycobot/joint7.dae; visual mesh filename=package://tork_moveit_tutorial/urdf/mycobot/joint7.dae

File: urdf/mycobot/withenv.urdf (robot description, URDF)
Before this commit: robot mycobot_ai_with, 9 links, 8 joints
Links:
- link env: geometry visual mesh filename=package://tork_moveit_tutorial/urdf/mycobot/suit_env.dae
- link joint1: geometry collision mesh filename=package://tork_moveit_tutorial/urdf/mycobot/joint1.dae; visual mesh filename=package://tork_moveit_tutorial/urdf/mycobot/joint1.dae
- link joint2: geometry collision mesh filename=package://tork_moveit_tutorial/urdf/mycobot/joint2.dae; visual mesh filename=package://tork_moveit_tutorial/urdf/mycobot/joint2.dae
- link joint3: geometry collision mesh filename=package://tork_moveit_tutorial/urdf/mycobot/joint3.dae; visual mesh filename=package://tork_moveit_tutorial/urdf/mycobot/joint3.dae
- link joint4: geometry collision mesh filename=package://tork_moveit_tutorial/urdf/mycobot/joint4.dae; visual mesh filename=package://tork_moveit_tutorial/urdf/mycobot/joint4.dae
- link joint5: geometry collision mesh filename=package://tork_moveit_tutorial/urdf/mycobot/joint5.stl; visual mesh filename=package://tork_moveit_tutorial/urdf/mycobot/joint5.stl
- link joint6: geometry collision mesh filename=package://tork_moveit_tutorial/urdf/mycobot/joint6.dae; visual mesh filename=package://tork_moveit_tutorial/urdf/mycobot/joint6.dae
- link joint6_flange: geometry collision mesh filename=package://tork_moveit_tutorial/urdf/mycobot/joint7.dae; visual mesh filename=package://tork_moveit_tutorial/urdf/mycobot/joint7.dae
